File: Schematics KiCad/Schematics KiCad.kicad_sch (KiCad schematic)
At the start: 11 parts, among them J1 OLED_128x64, J2 AHT20_Sensor, J3 Slide_Pot_Module, SW1 Start_Pause, SW2 Mode_Reset, U1 XIAO-RP2040-SMD

Commit message: Finished PCB design (footprints, layout, 3D models).
Parts:
- removed J1: OLED_128x64, Connector_PinSocket_2.54mm:PinSocket_1x04_P2.54mm_Vertical, symbol Connector_Generic:Conn_01x04
- removed J3: Slide_Pot_Module, Connector_PinSocket_2.54mm:PinSocket_1x03_P2.54mm_Horizontal, symbol Connector_Generic:Conn_01x03
- added RV1: R_Potentiometer, Potentiometer_THT:Potentiometer_Bourns_PTA6043_Single_Slide, symbol Device:R_Potentiometer
- added U2: OLED_128x64, Other_Components:MODULE_DM-OLED096-636, symbol DM-OLED096-636:DM-OLED096-636
Connections:
- net +3V3: now also RV1.3, U2.2 (VCC_IN)
- net GND: now also RV1.1, U2.1 (GND)
- net POT: now also RV1.2
- net SCL: now also U2.3 (SCL)
- net SDA: now also U2.4 (SDA)
